Commit message: added hardware interface

File: description/robot.urdf.xacro (robot description, xacro)
@@ -1,6 +1,13 @@
 <?xml version="1.0"?>
 <robot xmlns:xacro="https://www.ros.org/wiki/xacro" name="my_robot">
+    <xacro:arg name="use_ros2_control" default="true"/>
     <xacro:include filename="robot_body.xacro"/>
     <xacro:include filename="lidar.xacro"/>
-    <xacro:include filename="gazebo_control.xacro"/>
+    <xacro:include filename="camera.xacro"/>
+    <xacro:if value="$(arg use_ros2_control)">
+        <xacro:include filename="ros2_control.xacro"/>
+    </xacro:if>
+    <xacro:unless value="$(arg use_ros2_control)">
+        <xacro:include filename="gazebo_control.xacro"/>
+    </xacro:unless>
 </robot>

File: description/robot_body.xacro (robot description, xacro)
@@ -8,4 +8,7 @@
     <material name="black">
         <color rgba="0.0 0.0 0.0 1.0"/>
+    </material>
+    <material name="green">
+        <color rgba="0.0 1 0.0 1.0"/>
     </material>
     <!-- LINKS-->
