Commit message: added navigation

File: description/robot_body.xacro (robot description, xacro)
@@ -14,4 +14,5 @@
     <!-- LINKS-->
     <link name="base_link"></link>
+    <link name="base_footprint"></link>
     <link name="chassis">
         <visual>
@@ -126,4 +127,9 @@
     </gazebo>
     <!-- JOINTS-->
+    <joint name="base_footprint_joint" type="fixed">
+        <parent link="base_link"/>
+        <child link="base_footprint"/>
+        <origin xyz="0.0 0.0 0.0" rpy="0.0 0.0 0.0"/>
+    </joint>
     <joint name="chassis_joint" type="fixed">
         <parent link="base_link"/>
