Commit message: added amcl

File: description/lidar.xacro (robot description, xacro)
@@ -20,5 +20,5 @@
         <parent link="chassis"/>
         <child link="laser"/>
-        <origin xyz="0.2 0 0.32" rpy="0 0 0"/>
+        <origin xyz="0.2 0 0.28" rpy="0 0 0"/>
     </joint>
     <gazebo reference="laser">

File: description/ros2_control.xacro (robot description, xacro)
@@ -1,46 +1,4 @@
 <?xml version="1.0"?>
 <robot xmlns:xacro="https://www.ros.org/wiki/xacro">
-    <!-- <ros2_control name="GazeboSystem" type="system">
-        <hardware>
-            <plugin>gazebo_ros2_control/GazeboSystem</plugin>
-        </hardware>
-        <joint name="left_wheel_joint">
-            <command_interface name="velocity">
-                <param name="min">-10</param>
-                <param name="max">10</param>
-            </command_interface>
-            <state_interface name="velocity"/>
-            <state_interface name="position"/>
-        </joint>
-        <joint name="right_wheel_joint">
-            <command_interface name="velocity">
-                <param name="min">-10</param>
-                <param name="max">10</param>
-            </command_interface>
-            <state_interface name="velocity"/>
-            <state_interface name="position"/>
-        </joint>
-        <joint name="back_left_wheel_joint">
-            <command_interface name="velocity">
-                <param name="min">-10</param>
-                <param name="max">10</param>
-            </command_interface>
-            <state_interface name="velocity"/>
-            <state_interface name="position"/>
-        </joint>
-        <joint name="back_right_wheel_joint">
-            <command_interface name="velocity">
-                <param name="min">-10</param>
-                <param name="max">10</param>
-            </command_interface>
-            <state_interface name="velocity"/>
-            <state_interface name="position"/>
-        </joint>
-    </ros2_control>
-    <gazebo>
-        <plugin name="gazebo_ros2_control" filename="libgazebo_ros2_control.so">
-            <parameters>$(find my_robot)/config/my_controllers.yaml</parameters>
-        </plugin>
-    </gazebo> -->
     <ros2_control name="HardwareSystem" type="system">
         <hardware>
